File: poly88 backplane rev e/poly88 backplane rev e.kicad_pcb (KiCad board)
At the start: 2 copper layers, 31 parts, among them J1 Power In, J10 edge mount connector, J11 Conn_01x01, J2 Switch and Light, J3 Conn_01x01, J4 Card Edge in, J5 346-100-520-802, J6 346-100-520-802, J7 346-100-520-802, J8 346-100-520-802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

Commit message: components placed
Parts:
- added J12: Conn_01x01, Connector_Pin:Pin_D1.0mm_L10.0mm, F.Cu at (3.56, 44.1)
- added J13: Conn_01x01, Connector_Pin:Pin_D1.0mm_L10.0mm, F.Cu at (3.56, 35.9)
- added J14: Conn_01x01, Connector_Pin:Pin_D1.0mm_L10.0mm, F.Cu at (7.19, 12.1)
- added J15: Conn_01x01, Connector_Pin:Pin_D1.0mm_L10.0mm, F.Cu at (7.19, 17.1)
- added J16: Conn_01x01, Connector_Pin:Pin_D1.0mm_L10.0mm, F.Cu at (7.19, 22.2)
- moved R7 407.6 mm to (352.9, 3.15), turned to -90 degrees
- moved R6 391.0 mm to (349.1, 3.15), turned to -90 degrees
- moved Q1 328.1 mm to (353.3, 23.3)
- moved J2 323.4 mm to (360.3, 3.60), turned to -90 degrees
- moved R3 198.8 mm to (77.0, 36.7), turned to -90 degrees
- moved C4 183.8 mm to (68.2, 47.5), turned to 90 degrees
- moved R5 179.9 mm to (36.1, 46.3), turned to 180 degrees
- moved R4 179.4 mm to (36.1, 50.0), turned to 180 degrees
- moved R2 178.7 mm to (47.9, 40.0)
- moved R1 170.9 mm to (47.9, 44.5)
- moved D6 136.3 mm to (33.1, 2.04), turned to 180 degrees
- moved C2 133.9 mm to (5.48, 62.2)
- moved C1 133.6 mm to (80.5, 83.0), turned to 180 degrees
- moved J3 131.9 mm to (17.7, 35.4)
- moved J11 126.5 mm to (17.7, 43.8)
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- renumbered D2 to D1, D1 to D2, J3 to J11, J11 to J3
Connections:
- D1 pad 2: Net-(D2-Pad2) -> Net-(D1-Pad2)
- D2 pad 2: Net-(D1-Pad2) -> Net-(D2-Pad2)
- J1 pad 4: Net-(D2-Pad2) -> Net-(D1-Pad2)
- J1 pad 5: Net-(D1-Pad2) -> Net-(D2-Pad2)
- J11 pad 1: Net-(D3-Pad2) -> Net-(D1-Pad2)
- J2 pad 1: 1 -> Net-(J2-Pad1)
- J2 pad 3: Net-(J2-Pad3) -> 75
- J2 pad 4: 75 -> 1
- J3 pad 1: Net-(D1-Pad2) -> Net-(D2-Pad2)
- Q1 pad 3: Net-(J2-Pad3) -> Net-(J2-Pad1)
- R1 pad 1: 100 -> 2
- R1 pad 2: 2 -> 100
- R7 pad 2: Net-(J2-Pad3) -> Net-(J2-Pad1)
Other:
- board outline added: 365.1 x 102.7 mm
