File: poly88 backplane rev e/poly88 backplane rev e.kicad_sch (KiCad schematic)
At the start: 26 parts, among them J1 Power In, J11 Conn_01x01, J2 Switch and Light, J3 Conn_01x01, M1 Fan Option, Q1 2N5449

Commit message: components placed
Parts:
- added J? (x5): Conn_01x01, Connector_Pin:Pin_D1.0mm_L10.0mm, symbol Connector_Generic:Conn_01x01
Connections:
- net 1: now also J2.4 (Pin_4); no longer J2.1 (Pin_1)
- net 2: now also R1.1; no longer R1.2
- net 75: now also J2.3 (Pin_3); no longer J2.4 (Pin_4)
- net GND: now also R1.2, J?.1 (Pin_1), J?.1 (Pin_1), J?.1 (Pin_1); no longer R1.1
- net at D1.2 (A), J11.1 (Pin_1), R5.2: now also J1.4 (Pin_4), J?.1 (Pin_1); no longer J1.5 (Pin_5)
- net at D3.2 (A), D4.1 (K), J1.2 (Pin_2)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: no longer J3.1 (Pin_1)
- net at D2.2 (A): now also J1.5 (Pin_5), J3.1 (Pin_1), J?.1 (Pin_1); no longer J1.4 (Pin_4)
- net at Q1.3 (E), R7.2: now also J2.1 (Pin_1); no longer J2.3 (Pin_3)
Other:
- note added: "small change to schematic to match board layout"
