File: poly88 backplane rev 2.1/poly88 backplane rev 2.1.kicad_sch (KiCad schematic)
At the start: 28 parts, among them J1 Power In, J11 Conn_01x01, J12 Conn_01x01, J13 Conn_01x01, J2 Switch and Light, J3 Conn_01x01, M1 Fan Option, Q1 2N5449

Commit message: both layouts done?
Parts:
- added J14, J15, J16, J17, J18: Conn_01x01, Connector_Pin:Pin_D1.0mm_L10.0mm, symbol Connector_Generic:Conn_01x01
Connections:
- net 1: now also J17.1 (Pin_1); no longer J2.4 (Pin_4)
- net GND: now also J14.1 (Pin_1)
- net at D1.2 (A), J1.4 (Pin_4), J11.1 (Pin_1)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: now also J15.1 (Pin_1)
- net at D2.2 (A), J1.5 (Pin_5), J3.1 (Pin_1): now also J16.1 (Pin_1)
- new net: J18.1 (Pin_1), J2.4 (Pin_4)
Changed lines of the file:
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@@
   (junction (at 102.87 123.19) (diameter 0) (color 0 0 0 0)
   )
+  (junction (at 62.23 69.85) (diameter 0) (color 0 0 0 0)
+  )
   (junction (at 111.125 123.19) (diameter 0) (color 0 0 0 0)
   )
@@
   (junction (at 88.265 97.79) (diameter 0) (color 0 0 0 0)
   )
+  (junction (at 67.31 77.47) (diameter 0) (color 0 0 0 0)
+  )
   (junction (at 88.265 81.915) (diameter 0) (color 0 0 0 0)
   )
   (junction (at 104.775 110.49) (diameter 0) (color 0 0 0 0)
   )
+  (junction (at 37.465 62.23) (diameter 0) (color 0 0 0 0)
+  )
   (wire (pts (xy 118.745 114.3) (xy 190.5 114.3))
     (stroke (width 0) (type default) (color 0 0 0 0))
@@
     (stroke (width 0) (type default) (color 0 0 0 0))
   )
+  (wire (pts (xy 144.145 73.025) (xy 123.19 73.025))
+    (stroke (width 0) (type default) (color 0 0 0 0))
+  )
   (wire (pts (xy 118.745 121.92) (xy 118.745 123.19))
     (stroke (width 0) (type default) (color 0 0 0 0))
@@
     (stroke (width 0) (type default) (color 0 0 0 0))
   )
-  (wire (pts (xy 65.405 77.47) (xy 69.215 77.47))
+  (wire (pts (xy 65.405 77.47) (xy 67.31 77.47))
     (stroke (width 0) (type default) (color 0 0 0 0))
   )
@@
     (stroke (width 0) (type default) (color 0 0 0 0))
   )
+  (polyline (pts (xy 144.145 67.945) (xy 149.225 67.945))
+    (stroke (width 0) (type default) (color 0 0 0 0))
+  )
   (wire (pts (xy 153.035 78.105) (xy 153.035 85.725))
     (stroke (width 0) (type default) (color 0 0 0 0))
@@
     (stroke (width 0) (type default) (color 0 0 0 0))
   )
-  (wire (pts (xy 158.115 73.025) (xy 123.19 73.025))
+  (wire (pts (xy 158.115 73.025) (xy 149.225 73.025))
     (stroke (width 0) (type default) (color 0 0 0 0))
   )
@@
     (stroke (width 0) (type default) (color 0 0 0 0))
   )
+  (wire (pts (xy 37.465 62.23) (xy 41.91 62.23))
+    (stroke (width 0) (type default) (color 0 0 0 0))
+  )
   (wire (pts (xy 100.33 91.44) (xy 116.84 91.44))
+    (stroke (width 0) (type default) (color 0 0 0 0))
+  )
+  (wire (pts (xy 67.31 77.47) (xy 69.215 77.47))
     (stroke (width 0) (type default) (color 0 0 0 0))
   )
@@
     (pin "1")
   )
+  (symbol (lib_id "Connector_Generic:Conn_01x01") (at 41.91 57.15 90) (unit 1)
+    (in_bom yes) (on_board yes)
+    (property "Reference" "J14" (id 0) (at 38.735 55.88 90)
+      (effects (font (size 1.27 1.27)) (justify right))
+    )
+    (property "Value" "Conn_01x01" (id 1) (at 29.21 58.42 90)
+      (effects (font (size 1.27 1.27)) (justify right))
+    )
+    (property "Footprint" "Connector_Pin:Pin_D1.0mm_L10.0mm" (id 2) (at 41.91 57.15 0)
+      (effects (font (size 1.27 1.27)) hide)
+    )
+    (property "Datasheet" "~" (id 3) (at 41.91 57.15 0)
+      (effects (font (size 1.27 1.27)) hide)
+    )
+    (pin "1")
+  )
   (symbol (lib_id "Device:C_Polarized") (at 102.87 127 180) (unit 1)
     (in_bom yes) (on_board yes)
@@
     (pin "1")
   )
+  (symbol (lib_id "Connector_Generic:Conn_01x01") (at 144.145 67.945 90) (unit 1)
+    (in_bom yes) (on_board yes)
+    (property "Reference" "J17" (id 0) (at 140.97 66.675 90)
+      (effects (font (size 1.27 1.27)) (justify right))
+    )
+    (property "Value" "Conn_01x01" (id 1) (at 131.445 69.215 90)
+      (effects (font (size 1.27 1.27)) (justify right))
+    )
+    (property "Footprint" "Connector_Pin:Pin_D1.0mm_L10.0mm" (id 2) (at 144.145 67.945 0)
+      (effects (font (size 1.27 1.27)) hide)
+    )
+    (property "Datasheet" "~" (id 3) (at 144.145 67.945 0)
+      (effects (font (size 1.27 1.27)) hide)
+    )
+    (pin "1")
+  )
   (symbol (lib_id "power:GND") (at 99.695 64.135 0) (unit 1)
     (in_bom yes) (on_board yes) (fields_autoplaced)
@@
     (pin "1")
     (pin "2")
+  )
+  (symbol (lib_id "Connector_Generic:Conn_01x01") (at 67.31 72.39 90) (unit 1)
+    (in_bom yes) (on_board yes)
+    (property "Reference" "J16" (id 0) (at 64.135 72.39 90)
+      (effects (font (size 1.27 1.27)) (justify right))
+    )
+    (property "Value" "Conn_01x01" (id 1) (at 54.61 74.295 90)
+      (effects (font (size 1.27 1.27)) (justify right))
+    )
+    (property "Footprint" "Connector_Pin:Pin_D1.0mm_L10.0mm" (id 2) (at 67.31 72.39 0)
+      (effects (font (size 1.27 1.27)) hide)
+    )
+    (property "Datasheet" "~" (id 3) (at 67.31 72.39 0)
+      (effects (font (size 1.27 1.27)) hide)
+    )
+    (pin "1")
   )
   (symbol (lib_id "Device:C") (at 104.775 103.505 0) (unit 1)
@@
     (pin "1")
     (pin "2")
+  )
+  (symbol (lib_id "Connector_Generic:Conn_01x01") (at 149.225 67.945 90) (unit 1)
+    (in_bom yes) (on_board yes)
+    (property "Reference" "J18" (id 0) (at 146.05 66.675 90)
+      (effects (font (size 1.27 1.27)) (justify right))
+    )
+    (property "Value" "Conn_01x01" (id 1) (at 151.13 69.215 90)
+      (effects (font (size 1.27 1.27)) (justify right))
+    )
+    (property "Footprint" "Connector_Pin:Pin_D1.0mm_L10.0mm" (id 2) (at 149.225 67.945 0)
+      (effects (font (size 1.27 1.27)) hide)
+    )
+    (property "Datasheet" "~" (id 3) (at 149.225 67.945 0)
+      (effects (font (size 1.27 1.27)) hide)
+    )
+    (pin "1")
+  )
+  (symbol (lib_id "Connector_Generic:Conn_01x01") (at 57.15 69.85 180) (unit 1)
+    (in_bom yes) (on_board yes)
+    (property "Reference" "J15" (id 0) (at 53.34 68.58 0)
+      (effects (font (size 1.27 1.27)) (justify right))
+    )
+    (property "Value" "Conn_01x01" (id 1) (at 43.815 70.485 0)
+      (effects (font (size 1.27 1.27)) (justify right))
+    )
+    (property "Footprint" "Connector_Pin:Pin_D1.0mm_L10.0mm" (id 2) (at 57.15 69.85 0)
+      (effects (font (size 1.27 1.27)) hide)
+    )
+    (property "Datasheet" "~" (id 3) (at 57.15 69.85 0)
+      (effects (font (size 1.27 1.27)) hide)
+    )
+    (pin "1")
   )
   (symbol (lib_id "Connector_Generic:Conn_01x04") (at 163.195 75.565 0) (unit 1)
@@
       (reference "J13") (unit 1) (value "Conn_01x01") (footprint "Connector_Pin:Pin_D1.0mm_L10.0mm")
     )
+    (path "/25f53bfb-74b6-4ac1-a9b3-f0e5fcfb2acb"
+      (reference "J14") (unit 1) (value "Conn_01x01") (footprint "Connector_Pin:Pin_D1.0mm_L10.0mm")
+    )
+    (path "/e45f63fe-97a1-472d-9b2c-5df8bbe9a56c"
+      (reference "J15") (unit 1) (value "Conn_01x01") (footprint "Connector_Pin:Pin_D1.0mm_L10.0mm")
+    )
+    (path "/841da6f7-1698-4810-a4eb-50d82cc331bc"
+      (reference "J16") (unit 1) (value "Conn_01x01") (footprint "Connector_Pin:Pin_D1.0mm_L10.0mm")
+    )
+    (path "/6d481879-81c4-48e9-91e3-382a6573084e"
+      (reference "J17") (unit 1) (value "Conn_01x01") (footprint "Connector_Pin:Pin_D1.0mm_L10.0mm")
+    )
+    (path "/e1da2393-df63-4e7e-b7a4-ce89e3f149fc"
+      (reference "J18") (unit 1) (value "Conn_01x01") (footprint "Connector_Pin:Pin_D1.0mm_L10.0mm")
+    )
     (path "/0c058aee-43bf-4f42-94e9-66972df2f21c"
