File: poly88 backplane rev 2.1/poly88 backplane rev 2.1.kicad_pcb (KiCad board)
At the start: 2 copper layers, 365.1 x 102.7 mm, 33 parts, among them J1 Power In, J10 edge mount connector, J11 Conn_01x01, J12 Conn_01x01, J13 Conn_01x01, J2 Switch and Light, J3 Conn_01x01, J4 Card Edge in, J5 346-100-520-802, J6 346-100-520-802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

Commit message: both layouts done?
Parts:
- added J14: Conn_01x01, Connector_Pin:Pin_D1.0mm_L10.0mm, F.Cu at (7.24, 12.1)
- added J15: Conn_01x01, Connector_Pin:Pin_D1.0mm_L10.0mm, F.Cu at (7.24, 17.1)
- added J16: Conn_01x01, Connector_Pin:Pin_D1.0mm_L10.0mm, F.Cu at (7.24, 22.1)
- added J17: Conn_01x01, Connector_Pin:Pin_D1.0mm_L10.0mm, F.Cu at (353.3, 60.3)
- added J18: Conn_01x01, Connector_Pin:Pin_D1.0mm_L10.0mm, F.Cu at (353.3, 76.2)
Connections:
- J2 pad 4: 1 -> Net-(J2-Pad4)
Routing:
- net 48: track 177.9 -> 256.9 mm
- net Net-(J2-Pad4): track 0.00 -> 73.1 mm
- net 75: track 282.7 -> 341.5 mm
- net Net-(D1-Pad2): track 20.9 -> 67.2 mm
- net Net-(D2-Pad2): track 17.1 -> 42.9 mm
- net 1: track 396.7 -> 385.2 mm, vias 1 -> 2
- net 55: track 216.2 -> 220.2 mm
- net 100: track 182.7 -> 181.1 mm
Other:
- board text added: "1976"
- board text added: "60006"
- board text added: "BOTTOM"
- board text added: "BP/5 POLYMORPHIC SYSTEMS"
- board text added: "I.P.C."
- board text added: "R 2.1"
- board text removed: "101006 REV E BOTTOM"
- board text removed: "1977"
- board text removed: "Backplane 101006 REV E TOP"
- board text removed: "Interactive Products Corporation"
- board text removed: "PolyMorphic Systems"

Commit message: finished rev 2.1 pcb with annotations
Parts:
- added G***: LOGO, Evan's misc parts:OSHW gear, F.Cu at (41.2, 160.1)
- added G***: LOGO, Evan's misc parts:Evan Logo, F.Cu at (121.9, 99.2)
- moved C2 79.1 mm to (42.3, 132.2)
- moved C3 79.1 mm to (92.4, 88.8)
- moved C4 79.1 mm to (105.1, 117.5)
- moved D1 79.1 mm to (75.8, 109.2)
- moved D2 79.1 mm to (75.8, 102.8)
- moved D3 79.1 mm to (70.0, 87.8)
- moved D4 79.1 mm to (69.9, 83.1)
- moved D5 79.1 mm to (69.9, 76.2)
- moved D6 79.1 mm to (70.0, 72.0)
- moved D7 79.1 mm to (77.1, 120.0)
- moved D8 79.1 mm to (70.0, 92.5)
- moved J1 79.1 mm to (51.4, 77.0)
- moved J10 79.1 mm to (160.2, 60.8)
- moved J11 79.1 mm to (54.5, 113.7)
- moved J12 79.1 mm to (40.4, 114.1)
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Routing:
- net 1: track 385.2 -> 396.2 mm
Other:
- outline, holes or cut-outs redrawn
- board text added: "0vac"
- board text added: "1, 2, 51, and 52 do not connect between backplanes plugged into each other"
- board text added: "16vac"
- board text added: "71 is grounded here"
- board text added: "8v"
- board text added: "8vac"
- board text added: "Do Not Populate"
- board text added: "Poly88 pcb repro"
- board text added: "R4, R5, C4, D7 are for the RTC circuit only populate them on one backplane if you intend to connect multiple together"
- board text added: "TOP"
- board text added: "abzman2k.wordpress.com"
- board text added: "edge mount s100 connector here to chain chassis together"
- board text added: "fan connections soldered to 16vac pins on back (32v without center tap) smoothed with a cap it powers a nominally 24v fan"
- board text added: "gnd"
- board text added: "led"
- board text added: "rst"
